File: boardB/expansionboardB.kicad_pcb (KiCad board)
At the start: 2 copper layers, 131 x 83.8 mm, 51 parts, among them J1 USB_C_Receptacle, J3 HDMI_A, SW3 ESPRESET, SW4 ESPPROG, U1 ESP32-S3-WROOM-1, U2 GPIO_U2, U4 GPIO_U4, U5 SII1136CTU, U7 MAX20022ATIA+T

Commit message: Updates to new board
Parts:
- removed AU1: SJ-3523-SMT-TR, SJ-3523-SMT-TR:CUI_SJ-3523-SMT-TR
- removed C8, C9: 1uf, Capacitor_SMD:C_0603_1608Metric_Pad1.08x0.95mm_HandSolder
- removed R7, R8: 33Ohm, Resistor_SMD:R_0603_1608Metric_Pad0.98x0.95mm_HandSolder
- added C13: 2.2uf, Capacitor_SMD:C_0603_1608Metric_Pad1.08x0.95mm_HandSolder, B.Cu at (79.2, 77.0)
- C11, L3: moved to B.Cu
- moved C11 4.71 mm to (76.1, 78.5), turned to 180 degrees
- moved L3 4.46 mm to (76.2, 76.2)
- moved U5 3.74 mm to (123.9, 73.5)
- moved R9 3.68 mm to (135.3, 65.3)
- moved C12 1.05 mm to (82.0, 69.0)
Connections:
- L1 pad 1: /VOUT_1 -> REG3V3
- L2 pad 1: /VOUT_2 -> REG1V2
- L3 pad 2: /VOUT_3 -> REG1V0
- U5 pad 35: unconnected-(U5-SCK-Pad35) -> AU_SCLK
- U5 pad 36: unconnected-(U5-MCLK-Pad36) -> AU_MCLK
- U7 pad 15: unconnected-(U7-PV3-Pad15) -> 5V
- U7 pad 18: GND -> unconnected-(U7-PGND4-Pad18)
Routing:
- net REG3V3: track 68.0 -> 140.7 mm
- net REG1V2: track 12.4 -> 38.4 mm
- net REG1V0: track 0.00 -> 15.2 mm, vias 0 -> 1
- net 5V: track 180.0 -> 193.9 mm, vias 2 -> 11
- net D0_N: track 7.42 -> 20.1 mm, vias 0 -> 1
- net /PG_1: track 0.00 -> 12.6 mm, vias 0 -> 2
- net D0_P: track 7.64 -> 20.2 mm, vias 0 -> 1
- net AU_MCLK: track 12.0 -> 0.00 mm
- net AU_LRCLK: track 11.5 -> 0.00 mm
- net AU_SCLK: track 10.5 -> 0.00 mm
- net AU_SDIN: track 9.15 -> 0.00 mm
- net Net-(U7-LX3): track 0.00 -> 6.64 mm
- net Net-(AU1-Pad3): track 4.54 -> 0.00 mm
- net D2_P: track 11.4 -> 15.5 mm
- net D1_N: track 8.21 -> 12.3 mm
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Other:
- board text added: "1V0"

Commit message: Updated new board
Parts:
- removed C11: 10uf, Capacitor_SMD:C_0603_1608Metric_Pad1.08x0.95mm_HandSolder
- removed C13: 2.2uf, Capacitor_SMD:C_0603_1608Metric_Pad1.08x0.95mm_HandSolder
- removed D1: LED, LED_SMD:LED_1206_3216Metric_Pad1.42x1.75mm_HandSolder
- removed L3: 1.5uH, Inductor_SMD:L_0805_2012Metric
- added FB2: 1k@100MHz, Resistor_SMD:R_0805_2012Metric_Pad1.20x1.40mm_HandSolder, B.Cu at (93.4, 81.0)
- added FB3: 1k@100MHz, Resistor_SMD:R_0805_2012Metric_Pad1.20x1.40mm_HandSolder, B.Cu at (93.5, 66.4)
- added R13: 2K0, Resistor_SMD:R_0603_1608Metric_Pad0.98x0.95mm_HandSolder, B.Cu at (126.7, 57.7)
- added R14: 27K0, Resistor_SMD:R_0603_1608Metric_Pad0.98x0.95mm_HandSolder, B.Cu at (123.1, 61.1)
- added R7: 4K7, Resistor_SMD:R_0603_1608Metric_Pad0.98x0.95mm_HandSolder, B.Cu at (129.7, 58.9)
- added R8: 2K0, Resistor_SMD:R_0603_1608Metric_Pad0.98x0.95mm_HandSolder, B.Cu at (124.8, 57.7)
- added t1V2: 1V2_TEST, TestPoint:TestPoint_Pad_D1.5mm, B.Cu at (97.2, 81.0)
- added t3V3: 3V3_TEST, TestPoint:TestPoint_Pad_D1.5mm, B.Cu at (97.4, 66.5)
- added tSCL1: SCL_TEST, TestPoint:TestPoint_Pad_D1.5mm, B.Cu at (126.1, 53.8)
- added tSDA1: SDA_TEST, TestPoint:TestPoint_Pad_D1.5mm, B.Cu at (120.5, 58.5)
- R1, R10: value 23K -> 23K0
- R11, R12: value 10K -> 10K0
- R2: value 10KOhm -> 10K0
- R3, R4, R5, R6: value 33Ohm -> 33
- R9: value 510Ohm -> 4K06
- moved C10 2.19 mm to (93.3, 68.5), turned to 180 degrees
- moved C7 1.84 mm to (93.1, 79.0), turned to 180 degrees
- moved L1 1.46 mm to (91.1, 73.4), turned to 180 degrees
- moved R9 1.43 mm to (134.1, 66.0)
- moved L2 0.90 mm to (91.0, 75.3), turned to 180 degrees
Connections:
- C1 pad 1: REG3V3 -> /VOUT_1
- C6 pad 1: REG1V2 -> /VOUT_2
- CRD1 pad P1: GND -> SHLD
- CRD1 pad P2: GND -> SHLD
- CRD1 pad P3: GND -> SHLD
- CRD1 pad P4: GND -> SHLD
- J1 pad S1: GND -> SHLD
- J3 pad 13: unconnected-(J3-CEC-Pad13) -> D_CEC
- J3 pad 15: unconnected-(J3-SCL-Pad15) -> D_SCL
- J3 pad 16: unconnected-(J3-SDA-Pad16) -> D_SDA
- J3 pad 19: unconnected-(J3-HPD-Pad19) -> D_HPD
- L1 pad 1: REG3V3 -> /VOUT_1
- L2 pad 1: REG1V2 -> /VOUT_2
- R1 pad 1: REG3V3 -> /VOUT_1
- R10 pad 1: REG1V2 -> /VOUT_2
- R9 pad 2: REG3V3 -> GND
- U4 pad 17: AU_SDIN -> unconnected-(U4-Pin_17-Pad17)
- U4 pad 19: AU_SCLK -> unconnected-(U4-Pin_19-Pad19)
- U4 pad 21: AU_LRCLK -> unconnected-(U4-Pin_21-Pad21)
- U4 pad 23: AU_MCLK -> unconnected-(U4-Pin_23-Pad23)
- U4 pad 25: unconnected-(U4-Pin_25-Pad25) -> VR6
- U4 pad 26: unconnected-(U4-Pin_26-Pad26) -> VR7
- U4 pad 27: unconnected-(U4-Pin_27-Pad27) -> VR4
- U4 pad 28: unconnected-(U4-Pin_28-Pad28) -> VR5
- U4 pad 29: unconnected-(U4-Pin_29-Pad29) -> VR2
- U4 pad 30: unconnected-(U4-Pin_30-Pad30) -> VR3
- U4 pad 31: unconnected-(U4-Pin_31-Pad31) -> VR0
- U4 pad 32: unconnected-(U4-Pin_32-Pad32) -> VR1
- U4 pad 33: unconnected-(U4-Pin_33-Pad33) -> VG6
- U4 pad 34: unconnected-(U4-Pin_34-Pad34) -> VG7
- U4 pad 35: unconnected-(U4-Pin_35-Pad35) -> VG4
- U4 pad 36: unconnected-(U4-Pin_36-Pad36) -> VG5
- U4 pad 37: VDAT11 -> VG2
- U4 pad 38: VDAT10 -> VG3
- U4 pad 39: VDAT9 -> VG0
- U4 pad 40: VDAT8 -> VG1
- U4 pad 41: VDAT7 -> VB6
- U4 pad 42: VDAT6 -> VB7
- U4 pad 43: VDAT5 -> VB4
- U4 pad 44: VDAT4 -> VB5
- U4 pad 45: VDAT3 -> VB2
- U4 pad 46: VDAT2 -> VB3
- U4 pad 47: VDAT1 -> VB0
- U4 pad 48: VDAT0 -> VB1
- U4 pad 49: VCLK -> VVSYNC
- U4 pad 50: VDE -> VCLK
- U4 pad 51: VHSYNC -> VDE
- U4 pad 52: VVSYNC -> VHSYNC
- U4 pad 53: unconnected-(U4-Pin_53-Pad53) -> AU_SDIN
- U4 pad 54: unconnected-(U4-Pin_54-Pad54) -> AU_LRCLK
- U4 pad 55: unconnected-(U4-Pin_55-Pad55) -> AU_SCLK
- U4 pad 56: unconnected-(U4-Pin_56-Pad56) -> AU_MCLK
- U4 pad 57: unconnected-(U4-Pin_57-Pad57) -> VID_SCL
- U4 pad 58: unconnected-(U4-Pin_58-Pad58) -> VID_SDA
- U4 pad 59: unconnected-(U4-Pin_59-Pad59) -> VID_INT
- U4 pad 60: unconnected-(U4-Pin_60-Pad60) -> VID_RESETN
- U5 pad 10: unconnected-(U5-D8-Pad10) -> VB4
- U5 pad 11: unconnected-(U5-D7-Pad11) -> VB3
- U5 pad 13: unconnected-(U5-D6-Pad13) -> VB2
- U5 pad 14: unconnected-(U5-D5-Pad14) -> VB1
- U5 pad 15: unconnected-(U5-D4-Pad15) -> VB0
- U5 pad 17: unconnected-(U5-D3-Pad17) -> GND
- U5 pad 18: unconnected-(U5-D2-Pad18) -> GND
- U5 pad 19: unconnected-(U5-D1-Pad19) -> GND
- U5 pad 2: unconnected-(U5-D15-Pad2) -> GND
- U5 pad 20: unconnected-(U5-D0-Pad20) -> GND
- U5 pad 27: unconnected-(U5-DL3-Pad27) -> GND
- U5 pad 28: unconnected-(U5-DR3-Pad28) -> GND
- U5 pad 29: unconnected-(U5-SPDIF_IN_DL2-Pad29) -> GND
- U5 pad 3: unconnected-(U5-D14-Pad3) -> GND
- U5 pad 30: unconnected-(U5-SD3_DR2-Pad30) -> GND
- U5 pad 31: unconnected-(U5-SD2_DL1-Pad31) -> GND
- U5 pad 32: unconnected-(U5-SD1_DR1-Pad32) -> GND
- U5 pad 33: unconnected-(U5-SD0_DL0-Pad33) -> AU_SDIN
- U5 pad 34: unconnected-(U5-WS_DR0-Pad34) -> AU_LRCLK
- U5 pad 4: unconnected-(U5-D13-Pad4) -> GND
- U5 pad 40: unconnected-(U5-CEC_A-Pad40) -> D_CEC
- U5 pad 41: unconnected-(U5-DSDA-Pad41) -> D_SDA
- U5 pad 42: unconnected-(U5-DSCL-Pad42) -> D_SCL
- U5 pad 43: unconnected-(U5-CI2CA-Pad43) -> Net-(U5-CI2CA)
- U5 pad 44: unconnected-(U5-CSDA-Pad44) -> VID_SDA
- U5 pad 45: unconnected-(U5-CSCL-Pad45) -> VID_SCL
- U5 pad 46: AVINT -> VID_INT
- U5 pad 47: unconnected-(U5-~{RESET}-Pad47) -> VID_RESETN
- U5 pad 56: unconnected-(U5-AVCC-Pad56) -> REG1V2
- U5 pad 6: unconnected-(U5-D12-Pad6) -> GND
- U5 pad 61: unconnected-(U5-AVCC__1-Pad61) -> REG1V2
- U5 pad 7: unconnected-(U5-D11-Pad7) -> VB7
- U5 pad 76: unconnected-(U5-HPD-Pad76) -> D_HPD
- U5 pad 78: unconnected-(U5-D35-Pad78) -> VR7
- U5 pad 79: unconnected-(U5-D34-Pad79) -> VR6
- U5 pad 8: unconnected-(U5-D10-Pad8) -> VB6
- U5 pad 80: unconnected-(U5-D33-Pad80) -> VR5
- U5 pad 81: unconnected-(U5-D32-Pad81) -> VR4
- U5 pad 82: unconnected-(U5-D31-Pad82) -> VR3
- U5 pad 83: unconnected-(U5-D30-Pad83) -> VR2
- U5 pad 84: unconnected-(U5-D29-Pad84) -> VR1
- U5 pad 85: unconnected-(U5-D28-Pad85) -> VR0
- U5 pad 86: unconnected-(U5-D27-Pad86) -> GND
- U5 pad 87: unconnected-(U5-D26-Pad87) -> GND
- U5 pad 89: unconnected-(U5-D25-Pad89) -> GND
- U5 pad 9: unconnected-(U5-D9-Pad9) -> VB5
- U5 pad 90: unconnected-(U5-D24-Pad90) -> GND
- U5 pad 92: unconnected-(U5-D23-Pad92) -> VG7
- U5 pad 93: unconnected-(U5-D22-Pad93) -> VG6
- U5 pad 94: unconnected-(U5-D21-Pad94) -> VG5
- U5 pad 95: unconnected-(U5-D20-Pad95) -> VG4
- U5 pad 96: unconnected-(U5-D19-Pad96) -> VG3
- U5 pad 97: unconnected-(U5-D18-Pad97) -> VG2
- U5 pad 98: unconnected-(U5-D17-Pad98) -> VG1
- U5 pad 99: unconnected-(U5-D16-Pad99) -> VG0
- U7 pad 10: /PG_2 -> unconnected-(U7-PG2-Pad10)
- U7 pad 13: /PG_2 -> GND
- U7 pad 14: REG1V0 -> unconnected-(U7-OUTS3-Pad14)
- U7 pad 15: 5V -> unconnected-(U7-PV3-Pad15)
- U7 pad 16: Net-(U7-LX3) -> unconnected-(U7-LX3-Pad16)
- U7 pad 18: unconnected-(U7-PGND4-Pad18) -> GND
Routing:
- net 5V: track 193.9 -> 9.70 mm, vias 11 -> 4
- net REG3V3: track 140.7 -> 30.5 mm, vias 3 -> 8
- net Net-(D1-A): track 50.4 -> 0.00 mm, vias 1 -> 0
- net VID_RESETN: track 0.00 -> 40.4 mm
- net VID_INT: track 0.00 -> 37.0 mm
- net D_SCL: track 0.00 -> 36.4 mm, vias 0 -> 1
- net D_CEC: track 0.00 -> 34.6 mm, vias 0 -> 1
- net D_SDA: track 0.00 -> 31.7 mm, vias 0 -> 1
- net VID_SDA: track 0.00 -> 30.8 mm, vias 0 -> 1
- net VID_SCL: track 0.00 -> 29.6 mm, vias 0 -> 1
- net VR7: track 0.00 -> 28.3 mm
- net D_HPD: track 0.00 -> 27.2 mm, vias 0 -> 1
- net VR5: track 0.00 -> 26.2 mm
- net VR3: track 0.00 -> 25.3 mm
- net VR1: track 0.00 -> 24.4 mm
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- added copper zone on In2.Cu, net 5V
- added copper zone on In1.Cu, net GND
- added copper zone on In2.Cu, net GND
- added copper zone on In2.Cu, net REG1V2
- added copper zone on In2.Cu, net REG3V3
- added copper zone on In2.Cu, net SHLD
Other:
- copper layers 2 -> 4
- board text added: "tinysys issue 3A December 2025 Engin Cilasun"
- board text removed: "1V0"
- board text removed: "1V2"
- board text removed: "3V3"
- board text removed: "3v3"
- board text removed: "5v0"
- board text removed: "AA1"
- board text removed: "AA19"
- board text removed: "AA20"
- board text removed: "AA3"
- board text removed: "AB1"
- board text removed: "AB2"
- board text removed: "AB21"
- board text removed: "AB3"
- board text removed: "GND"
- board text removed: "H2"
- board text removed: "K1"
- board text removed: "K2"
- board text removed: "M1"
- board text removed: "N17"
- board text removed: "POWER"
- board text removed: "R18"
- board text removed: "R4"
- board text removed: "T1"
- board text removed: "T21"
- board text removed: "T4"
- board text removed: "T5"
- board text removed: "U1"
- board text removed: "U17"
- board text removed: "U20"
- board text removed: "U5"
- board text removed: "V18"
- board text removed: "V4"
- board text removed: "VCC"
- board text removed: "W1"
- board text removed: "W4"
- board text removed: "Y1"
- board text removed: "Y18"
- board text removed: "Y21"
- board text removed: "Y3"
- board text removed: "tinysys issue 2G December 2024 Engin Cilasun"

Commit message: Updates to new board
Parts:
- added E1: SparkGap, Diode_SMD:D_0201_0603Metric, F.Cu at (23.9, 82.5)
- added E1: SparkGap, Diode_SMD:D_0201_0603Metric, F.Cu at (144.6, 120.5)
- added E1: SparkGap, Diode_SMD:D_0201_0603Metric, F.Cu at (144.6, 44.5)
- added E1: SparkGap, Diode_SMD:D_0201_0603Metric, F.Cu at (30.9, 44.5)
- added E1: SparkGap, Diode_SMD:D_0201_0603Metric, F.Cu at (31.0, 120.5)
- REF** (x4): moved to F.Cu
- moved REF** 24.5 mm to (119.0, 109.7), turned to 0 degrees
- moved REF** 16.2 mm to (122.1, 102.0), turned to 0 degrees
- moved REF** 13.7 mm to (125.5, 109.2), turned to 0 degrees
- moved REF** 8.92 mm to (131.4, 109.2), turned to 0 degrees
- moved C7 2.19 mm to (95.3, 79.1), turned to 0 degrees
- moved t1V2 2.05 mm to (98.5, 82.6)
- moved t3V3 2.04 mm to (98.5, 64.8)
- moved C10 2.01 mm to (95.3, 68.5), turned to 0 degrees
- moved L1 1.52 mm to (91.1, 71.9)
- moved L2 0.89 mm to (91.0, 76.2)
- moved FB2 0.16 mm to (93.5, 81.0)
- moved R10 0.10 mm to (89.6, 81.0)
Connections:
- U4 pad 14: GPI -> unconnected-(U4-Pin_14-Pad14)
Routing:
- net SHLD: track 24.0 -> 37.8 mm
- net 5V: track 9.70 -> 17.2 mm
- net REG1V2: track 20.4 -> 22.5 mm
- net /VOUT_1: track 13.6 -> 11.7 mm
- net REG3V3: track 30.5 -> 32.2 mm
- net /VOUT_2: track 12.2 -> 10.8 mm
- net Net-(U7-LX1): track 3.84 -> 4.47 mm
- net GND: vias 46 -> 37
Other:
- board text added: "Designed by Engin Cilasun Model E001 January 2025 https://github.com/ecilasun/tinysys WARNING: PROTOTYPE DEVICE"
- board text removed: "tinysys issue 3A December 2025 Engin Cilasun"

Commit message: Updated board and hardware to reset ESP32 from the FPGA
Parts:
- removed SW3: ESPRESET, Button_Switch_SMD:SW_Tactile_SPST_NO_Straight_CK_PTS636Sx25SMTRLFS
Connections:
- C4 pad 1: Net-(U1-EN) -> ESP_RST
- R2 pad 1: Net-(U1-EN) -> ESP_RST
- U1 pad 3: Net-(U1-EN) -> ESP_RST
- U2 pad 60: unconnected-(U2-Pin_60-Pad60) -> ESP_RST
Routing:
- net ESP_RST: track 0.00 -> 51.3 mm, vias 0 -> 1
- net Net-(U1-EN): track 22.9 -> 0.00 mm
Other:
- board text removed: "RESET"

Commit message: minor repairs to boot time
Routing:
- net CK_P: track 12.2 -> 21.3 mm
- net CK_N: track 12.2 -> 21.3 mm
- net D1_P: track 12.3 -> 21.3 mm
- net D1_N: track 12.3 -> 21.3 mm
- net D2_P: track 15.5 -> 21.3 mm
- net D2_N: track 15.5 -> 21.3 mm
- net REG3V3: track 32.2 -> 30.3 mm, vias 8 -> 7

Commit message: New board updates
Parts:
- added JTAG1: Conn_01x06_Pin, Connector_PinHeader_2.54mm:PinHeader_1x06_P2.54mm_Vertical, F.Cu at (131.4, 120.0)
Connections:
- U1 pad 18: unconnected-(U1-IO10-Pad18) -> IO10
- U1 pad 19: unconnected-(U1-IO11-Pad19) -> IO11
- U1 pad 20: unconnected-(U1-IO12-Pad20) -> IO12
- U1 pad 21: unconnected-(U1-IO13-Pad21) -> IO13
- U1 pad 22: unconnected-(U1-IO14-Pad22) -> IO22
- U1 pad 23: unconnected-(U1-IO21-Pad23) -> IO21
- U1 pad 24: unconnected-(U1-IO47-Pad24) -> IO47
- U1 pad 25: unconnected-(U1-IO48-Pad25) -> IO48
- U2 pad 33: unconnected-(U2-Pin_33-Pad33) -> IO10
- U2 pad 35: unconnected-(U2-Pin_35-Pad35) -> IO11
- U2 pad 37: unconnected-(U2-Pin_37-Pad37) -> IO12
- U2 pad 39: unconnected-(U2-Pin_39-Pad39) -> IO13
- U2 pad 41: unconnected-(U2-Pin_41-Pad41) -> IO22
- U2 pad 43: unconnected-(U2-Pin_43-Pad43) -> IO21
- U2 pad 45: unconnected-(U2-Pin_45-Pad45) -> IO47
- U2 pad 47: unconnected-(U2-Pin_47-Pad47) -> IO48
- U4 pad 11: unconnected-(U4-Pin_11-Pad11) -> TDO
- U4 pad 13: unconnected-(U4-Pin_13-Pad13) -> TCK
- U4 pad 7: unconnected-(U4-Pin_7-Pad7) -> TMS
- U4 pad 9: unconnected-(U4-Pin_9-Pad9) -> TDI
Routing:
- net IO10: track 0.00 -> 28.4 mm
- net TCK: track 0.00 -> 26.5 mm
- net TDO: track 0.00 -> 26.4 mm
- net TDI: track 0.00 -> 26.3 mm
- net TMS: track 0.00 -> 26.3 mm
- net IO11: track 0.00 -> 25.6 mm
- net IO12: track 0.00 -> 22.8 mm
- net IO13: track 0.00 -> 20.1 mm
- net IO22: track 0.00 -> 17.5 mm
- net IO21: track 0.00 -> 14.9 mm
- net IO47: track 0.00 -> 12.9 mm
- net IO48: track 0.00 -> 9.83 mm
- net unconnected-(U2-Pin_45-Pad45): track 0.52 -> 0.00 mm
- net GND: vias 37 -> 36
