File: boardB/expansionboardB.kicad_sch (KiCad schematic)
At the start: 46 parts, among them J1 USB_C_Receptacle, J3 HDMI_A, SW4 ESPPROG, U1 ESP32-S3-WROOM-1, U2 GPIO_U2, U4 GPIO_U4, U5 SII1136CTU, U7 MAX20022ATIA+T, t1V2 1V2_TEST, t3V3 3V3_TEST

Commit message: Resistor mistake
Parts:
- R10: value 23K0 -> 2K0
- R9: value 4K06 -> 4K02
Other:
- note added: "1V2 -> R10=R11*0.2 R10==2KOhm R11==10KOhm C6==75pF"
- note added: "2V5 -> Ra=Rb*1.5 Ra==15KOhm Rb==10KOhm Ca==15pF"
- note added: "3V3 -> R1=R12*2.3 R1==23KOhm R12==10KOhm C1==15pF"
- note added: "5V0 -> Ra=Rb*4.0 Ra==40KOhm Rb==10KOhm Ca==15pF"
- note added: "CAN'T FIND THIS!"
- note removed: "1V2 -> R1=R2*0.2 R1==2KOhm R2==10KOhm C1==75pF"
- note removed: "2V5 -> R1=R2*1.5 R1==15KOhm R2==10KOhm C1==15pF"
- note removed: "3V3 -> R1=R2*2.3 R1==23KOhm R2==10KOhm C1==15pF"
- note removed: "5V0 -> R1=R2*4.0 R1==40KOhm R2==10KOhm C1==15pF"
Changed lines of the file:
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@@
 		)
 	)
-	(text "5V0 -> R1=R2*4.0\nR1==40KOhm\nR2==10KOhm\nC1==15pF"
+	(text "5V0 -> Ra=Rb*4.0\nRa==40KOhm\nRb==10KOhm\nCa==15pF"
 		(exclude_from_sim no)
 		(at 288.29 243.84 0)
@@
 		)
 	)
-	(text "3V3 -> R1=R2*2.3\nR1==23KOhm\nR2==10KOhm\nC1==15pF"
+	(text "3V3 -> R1=R12*2.3\nR1==23KOhm\nR12==10KOhm\nC1==15pF"
 		(exclude_from_sim no)
 		(at 288.29 233.172 0)
@@
 		)
 	)
-	(text "2V5 -> R1=R2*1.5\nR1==15KOhm\nR2==10KOhm\nC1==15pF"
+	(text "2V5 -> Ra=Rb*1.5\nRa==15KOhm\nRb==10KOhm\nCa==15pF"
 		(exclude_from_sim no)
 		(at 288.29 238.506 0)
@@
 		)
 	)
-	(text "1V2 -> R1=R2*0.2\nR1==2KOhm\nR2==10KOhm\nC1==75pF"
+	(text "1V2 -> R10=R11*0.2\nR10==2KOhm\nR11==10KOhm\nC6==75pF"
 		(exclude_from_sim no)
 		(at 288.29 227.838 0)
@@
 		)
 	)
+	(text "CAN'T FIND THIS!"
+		(exclude_from_sim no)
+		(at 227.584 241.808 0)
+		(effects
+			(font
+				(size 0.762 0.762)
+			)
+			(justify left)
+		)
+	)
 	(text "640x480 (480p)\nITU-R BT.601\nY = 0.299R′ + 0.587G′ + 0.114B′ \nCb = –0.172R′ – 0.339G′ + 0.511B′ + 128 \nCr = 0.511R′ – 0.428G′ – 0.083B′ + 128"
 		(exclude_from_sim no)
@@
 			)
 		)
-		(property "Value" "23K0"
-			(at 237.49 241.554 0)
+		(property "Value" "2K0"
+			(at 238.506 241.554 0)
 			(effects
 				(font
@@
 			)
 		)
-		(property "Value" "4K06"
+		(property "Value" "4K02"
 			(at 147.574 155.194 90)
 			(effects

Commit message: Board updates
Parts:
- added R15: 10K0, Resistor_SMD:R_0603_1608Metric_Pad0.98x0.95mm_HandSolder, symbol Device:R
- added R16: 3K0, Resistor_SMD:R_0603_1608Metric_Pad0.98x0.95mm_HandSolder, symbol Device:R
- R1: value 23K0 -> 10K0
Connections:
- net VOUT_1: now also R16.1; no longer R1.1
- new net: R15.1, R16.2
- new net: R1.1, R15.2
Other:
- note removed: "CAN'T FIND THIS!"
- moved on the sheet: R1, R12
